File: receiver_485/ReceiverRS485.kicad_pcb (KiCad board)
At the start: 2 copper layers, 69.2 x 100 mm, 93 parts, among them J1 USB3_A, J10 USB3_duplo, J2 Conn_01x03, J3 USB3_A, J4 Conn_01x03, J5 USB3_A, J6 Conn_01x03, J7 USB3_A, J8 Conn_01x03, J9 USB3_duplo, U1 RFM-0505S, U10 MAX3283E, U11 TLP2372, U12 TLP2372, U13 RFM-0505S, U14 MAX3283E, U15 TLP2372, U16 MAX3283E, U17 TLP2372, U18 TLP2372, U19 RFM-0505S, U2 MAX3283E, U20 MAX3283E, U21 TLP2372, U22 MAX3283E, U23 TLP2372, U24 TLP2372, U3 TLP2372, U4 MAX3283E, U5 TLP2372, U6 TLP2372, U7 RFM-0505S, U8 MAX3283E, U9 TLP2372

Commit message: USB position
Parts:
- moved J9 0.35 mm to (111.3, 59.1)
- moved J10 0.33 mm to (111.3, 120.0)
Routing:
- net D+_ch4: track 116.6 -> 118.6 mm
- net D+_ch1: track 133.5 -> 135.4 mm
- net D-_ch1: track 60.2 -> 61.9 mm
- net drain_ch1: track 45.1 -> 46.5 mm
- net D+_ch2: track 120.4 -> 121.7 mm
- net sstx+_ch1: track 24.1 -> 25.0 mm
- net sstx+_ch2: track 31.6 -> 32.4 mm
- net sstx+_ch4: track 18.2 -> 18.9 mm
- net sstx-_ch2: track 30.4 -> 31.1 mm
- net sstx-_ch1: track 31.6 -> 32.2 mm
- net ssrx+_ch3: track 57.8 -> 57.3 mm
