File: Panel/RearPanel.kicad_pcb (KiCad board)
At the start: 2 copper layers, 103 x 53 mm, 4 parts

Commit message: Panel update
Other:
- board text added: "Channel 1"
- board text added: "Channel 2"
- board text added: "Channel 3"
- board text added: "Channel 4"
- board text added: "Iot Group - 2021"
Changed lines of the file:
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@@
   (general
     (thickness 1.6)
-    (drawings 49)
+    (drawings 54)
     (tracks 0)
     (zones 0)
@@
     )
   )
+  (gr_text "Iot Group - 2021" (at 151.07724 114.69084) (layer F.SilkS)
+    (effects (font (size 1 1) (thickness 0.15)))
+  )
+  (gr_text "Channel 4" (at 147.77724 90.36084) (layer F.SilkS)
+    (effects (font (size 1 1) (thickness 0.15)))
+  )
+  (gr_text "Channel 3" (at 147.77724 70.57084) (layer F.SilkS)
+    (effects (font (size 1 1) (thickness 0.15)))
+  )
+  (gr_text "Channel 2" (at 87.26724 90.36084) (layer F.SilkS)
+    (effects (font (size 1 1) (thickness 0.15)))
+  )
+  (gr_text "Channel 1" (at 87.26724 70.55084) (layer F.SilkS)
+    (effects (font (size 1 1) (thickness 0.15)))
+  )
   (gr_line (start 155.12724 72.56084) (end 140.42724 72.56084) (layer Edge.Cuts) (width 0.15))
